File: pcb/usb_pd_board.kicad_sch (KiCad schematic)
At the start: 30 parts, among them J1 USB_C_Receptacle, Q1 SI7141DP-T1-GE3, U1 STUSB4500QTR, U2 AP63203WU

Commit message: datenblätter
Parts:
- added C10, C11, C12, C13, C18: 100nF, Capacitor_SMD:C_0603_1608Metric_Pad1.08x0.95mm_HandSolder, symbol Device:C_Small
- added C14: 10uF, Capacitor_SMD:C_0402_1005Metric_Pad0.74x0.62mm_HandSolder, symbol Device:C_Small
- added C15: 10nF, Capacitor_SMD:C_0603_1608Metric_Pad1.08x0.95mm_HandSolder, symbol Device:C_Small
- added C16, C17: 1uF, Capacitor_SMD:C_0603_1608Metric_Pad1.08x0.95mm_HandSolder, symbol Device:C_Small
- added FB1: 120R, Inductor_SMD:L_0402_1005Metric_Pad0.77x0.64mm_HandSolder, symbol Device:FerriteBead
- added R11: 10k, Resistor_SMD:R_0402_1005Metric_Pad0.72x0.64mm_HandSolder, symbol Device:R_Small
- added U3: STM32F103C8Tx, Package_QFP:LQFP-48_7x7mm_P0.5mm, symbol MCU_ST_STM32F1:STM32F103C8Tx
Connections:
- net +3.3V: now also C10.2, C11.2, C12.2, C13.2, C14.1, C17.2, FB1.2, U3.1 (VBAT), U3.24 (VDD), U3.36 (VDD), U3.48 (VDD)
- net GND: now also C10.1, C11.1, C12.1, C13.1, C14.2, C15.1, C16.1, C17.1, C18.1, U3.23 (VSS), U3.35 (VSS), U3.47 (VSS), U3.8 (VSSA)
- new net: C18.2, U3.7 (NRST)
- new net: R11.2, U3.44 (BOOT0)
- new net +3.3VA: C15.2, C16.2, FB1.1, U3.9 (VDDA)
Other:
- note added: "Decoupling STM32"
- moved on the sheet: C4, C5, C6, C7, Q1, R10, R3, R4, R7, R8, R9, U1
